File: power_board/power_board.kicad_sch (KiCad schematic)
At the start: 14 parts, among them J1 AC2, J2 AC3, J3 AC1, J4 VCCB, J5 VCCA

Commit message: redesigned the power loop
Parts:
- removed J4: VCCB, Connector_PinHeader_2.54mm:PinHeader_2x04_P2.54mm_Vertical, symbol Connector_Generic:Conn_02x04_Odd_Even
- removed J5: VCCA, Connector_PinHeader_2.54mm:PinHeader_2x04_P2.54mm_Vertical, symbol Connector_Generic:Conn_02x04_Odd_Even
- added H1, H2, H3, H4: MountingHole, MountingHole:MountingHole_3.2mm_M3, symbol Mechanical:MountingHole
- added J4: Conn_01x06_Male, Connector_PinHeader_1.27mm:PinHeader_1x06_P1.27mm_Horizontal, symbol Connector:Conn_01x06_Male
Connections:
- net at PS2.5 (+VOUT): now also J4.3 (Pin_3)
- net at PS2.4 (-VOUT): now also J4.4 (Pin_4)
- net at PS3.4 (-VOUT): now also J4.6 (Pin_6)
- net at PS3.5 (+VOUT): now also J4.5 (Pin_5)
- net at PS1.2 (-VOUT): now also J4.2 (Pin_2)
- net at PS1.3 (+VOUT): now also J4.1 (Pin_1)
- no-connect marks 4 -> 0

Commit message: Updated final design
Parts:
- removed J4: Conn_01x06_Male, Connector_PinHeader_1.27mm:PinHeader_1x06_P1.27mm_Horizontal, symbol Connector:Conn_01x06_Male
- added J4: Conn_02x05_Odd_Even, 61201021621:SHDR10W64P254_2X5_2036X885X925P, symbol Connector_Generic:Conn_02x05_Odd_Even
Connections:
- net at PS3.4 (-VOUT): now also J4.5 (Pin_5)
- net at PS3.5 (+VOUT): now also J4.6 (Pin_6)
- net at PS1.3 (+VOUT): now also J4.2 (Pin_2)
- net at PS1.2 (-VOUT): now also J4.1 (Pin_1)
- net at PS2.5 (+VOUT): now also J4.4 (Pin_4)
- net at PS2.4 (-VOUT): now also J4.3 (Pin_3)
- no-connect marks 0 -> 4
Changed lines of the file:
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@@
 (kicad_sch (version 20211123) (generator eeschema)
   (paper "A4")
+  (no_connect (at 149.86 81.28))
+  (no_connect (at 149.86 83.82))
+  (no_connect (at 162.56 83.82))
+  (no_connect (at 162.56 81.28))
   (wire (pts (xy 74.295 102.87) (xy 81.28 102.87))
     (stroke (width 0) (type default) (color 0 0 0 0))
   )
-  (wire (pts (xy 133.35 58.42) (xy 133.35 73.66))
+  (wire (pts (xy 118.745 80.01) (xy 130.81 80.01))
     (stroke (width 0) (type default) (color 0 0 0 0))
   )
@@
     (stroke (width 0) (type default) (color 0 0 0 0))
   )
+  (wire (pts (xy 162.56 58.42) (xy 162.56 73.66))
+    (stroke (width 0) (type default) (color 0 0 0 0))
+  )
+  (wire (pts (xy 129.54 74.93) (xy 162.56 74.93))
+    (stroke (width 0) (type default) (color 0 0 0 0))
+  )
   (wire (pts (xy 117.475 60.96) (xy 131.445 60.96))
     (stroke (width 0) (type default) (color 0 0 0 0))
   )
-  (wire (pts (xy 131.445 60.96) (xy 131.445 76.2))
+  (wire (pts (xy 131.445 60.96) (xy 131.445 73.66))
     (stroke (width 0) (type default) (color 0 0 0 0))
   )
@@
     (stroke (width 0) (type default) (color 0 0 0 0))
   )
-  (wire (pts (xy 118.745 81.28) (xy 148.59 81.28))
-    (stroke (width 0) (type default) (color 0 0 0 0))
-  )
-  (wire (pts (xy 129.54 83.82) (xy 148.59 83.82))
-    (stroke (width 0) (type default) (color 0 0 0 0))
-  )
   (wire (pts (xy 118.745 79.375) (xy 129.54 79.375))
     (stroke (width 0) (type default) (color 0 0 0 0))
@@
     (stroke (width 0) (type default) (color 0 0 0 0))
   )
-  (wire (pts (xy 131.445 86.36) (xy 148.59 86.36))
-    (stroke (width 0) (type default) (color 0 0 0 0))
-  )
-  (wire (pts (xy 129.54 79.375) (xy 129.54 78.74))
+  (wire (pts (xy 129.54 79.375) (xy 129.54 74.93))
+    (stroke (width 0) (type default) (color 0 0 0 0))
+  )
+  (wire (pts (xy 131.445 81.915) (xy 133.985 81.915))
     (stroke (width 0) (type default) (color 0 0 0 0))
   )
@@
     (stroke (width 0) (type default) (color 0 0 0 0))
   )
-  (wire (pts (xy 129.54 100.33) (xy 129.54 83.82))
-    (stroke (width 0) (type default) (color 0 0 0 0))
-  )
-  (wire (pts (xy 133.35 73.66) (xy 148.59 73.66))
+  (wire (pts (xy 129.54 100.33) (xy 129.54 81.28))
+    (stroke (width 0) (type default) (color 0 0 0 0))
+  )
+  (wire (pts (xy 130.81 76.2) (xy 130.81 80.01))
     (stroke (width 0) (type default) (color 0 0 0 0))
   )
@@
     (stroke (width 0) (type default) (color 0 0 0 0))
   )
-  (wire (pts (xy 129.54 78.74) (xy 148.59 78.74))
-    (stroke (width 0) (type default) (color 0 0 0 0))
-  )
-  (wire (pts (xy 131.445 76.2) (xy 148.59 76.2))
+  (wire (pts (xy 131.445 73.66) (xy 149.86 73.66))
+    (stroke (width 0) (type default) (color 0 0 0 0))
+  )
+  (wire (pts (xy 149.86 76.2) (xy 130.81 76.2))
     (stroke (width 0) (type default) (color 0 0 0 0))
   )
@@
     (stroke (width 0) (type default) (color 0 0 0 0))
   )
-  (wire (pts (xy 118.745 81.28) (xy 118.745 81.915))
-    (stroke (width 0) (type default) (color 0 0 0 0))
-  )
-  (wire (pts (xy 131.445 102.87) (xy 131.445 86.36))
+  (wire (pts (xy 129.54 81.28) (xy 132.715 81.28))
+    (stroke (width 0) (type default) (color 0 0 0 0))
+  )
+  (wire (pts (xy 162.56 77.47) (xy 162.56 78.74))
+    (stroke (width 0) (type default) (color 0 0 0 0))
+  )
+  (wire (pts (xy 118.745 80.01) (xy 118.745 81.915))
+    (stroke (width 0) (type default) (color 0 0 0 0))
+  )
+  (wire (pts (xy 131.445 81.915) (xy 131.445 102.87))
     (stroke (width 0) (type default) (color 0 0 0 0))
   )
@@
     (stroke (width 0) (type default) (color 0 0 0 0))
   )
-  (wire (pts (xy 117.475 58.42) (xy 133.35 58.42))
+  (wire (pts (xy 132.715 81.28) (xy 132.715 77.47))
+    (stroke (width 0) (type default) (color 0 0 0 0))
+  )
+  (wire (pts (xy 133.985 78.74) (xy 133.985 81.915))
+    (stroke (width 0) (type default) (color 0 0 0 0))
+  )
+  (wire (pts (xy 133.985 78.74) (xy 149.86 78.74))
+    (stroke (width 0) (type default) (color 0 0 0 0))
+  )
+  (wire (pts (xy 132.715 77.47) (xy 162.56 77.47))
+    (stroke (width 0) (type default) (color 0 0 0 0))
+  )
+  (wire (pts (xy 162.56 74.93) (xy 162.56 76.2))
+    (stroke (width 0) (type default) (color 0 0 0 0))
+  )
+  (wire (pts (xy 117.475 58.42) (xy 162.56 58.42))
     (stroke (width 0) (type default) (color 0 0 0 0))
   )
@@
     (pin "2")
   )
-  (symbol (lib_id "Connector:Conn_01x06_Male") (at 153.67 78.74 0) (mirror y) (unit 1)
-    (in_bom yes) (on_board yes) (fields_autoplaced)
-    (property "Reference" "J4" (id 0) (at 154.94 78.7399 0)
-      (effects (font (size 1.27 1.27)) (justify right))
-    )
-    (property "Value" "Conn_01x06_Male" (id 1) (at 154.94 81.2799 0)
-      (effects (font (size 1.27 1.27)) (justify right))
-    )
-    (property "Footprint" "Connector_PinHeader_1.27mm:PinHeader_1x06_P1.27mm_Horizontal" (id 2) (at 153.67 78.74 0)
-      (effects (font (size 1.27 1.27)) hide)
-    )
-    (property "Datasheet" "~" (id 3) (at 153.67 78.74 0)
-      (effects (font (size 1.27 1.27)) hide)
-    )
-    (pin "1")
+  (symbol (lib_id "Connector_Generic:Conn_02x05_Odd_Even") (at 154.94 78.74 0) (unit 1)
+    (in_bom yes) (on_board yes) (fields_autoplaced)
+    (property "Reference" "J4" (id 0) (at 156.21 67.31 0))
+    (property "Value" "Conn_02x05_Odd_Even" (id 1) (at 156.21 69.85 0))
+    (property "Footprint" "61201021621:SHDR10W64P254_2X5_2036X885X925P" (id 2) (at 154.94 78.74 0)
+      (effects (font (size 1.27 1.27)) hide)
+    )
+    (property "Datasheet" "~" (id 3) (at 154.94 78.74 0)
+      (effects (font (size 1.27 1.27)) hide)
+    )
+    (pin "1")
+    (pin "10")
     (pin "2")
     (pin "3")
@@
     (pin "5")
     (pin "6")
+    (pin "7")
+    (pin "8")
+    (pin "9")
   )
   (symbol (lib_id "Mechanical:MountingHole") (at 88.265 140.335 90) (unit 1)
@@
       (reference "J3") (unit 1) (value "AC1") (footprint "Connector_Molex:Molex_KK-396_A-41791-0002_1x02_P3.96mm_Vertical")
     )
-    (path "/543caa26-976e-4e09-a9ff-48a5f70c6099"
-      (reference "J4") (unit 1) (value "Conn_01x06_Male") (footprint "Connector_PinHeader_1.27mm:PinHeader_1x06_P1.27mm_Horizontal")
+    (path "/73c4d883-0af7-4246-841b-b05544b5be1f"
+      (reference "J4") (unit 1) (value "Conn_02x05_Odd_Even") (footprint "61201021621:SHDR10W64P254_2X5_2036X885X925P")
     )
     (path "/da58b535-f243-4501-ade6-853032d8d15b"

Commit message: Final design
Parts:
- removed J4: Conn_02x05_Odd_Even, 61201021621:SHDR10W64P254_2X5_2036X885X925P, symbol Connector_Generic:Conn_02x05_Odd_Even
- added J4: Conn_02x03_Odd_Even, Connector_PinHeader_2.54mm:PinHeader_2x03_P2.54mm_Horizontal, symbol Connector_Generic:Conn_02x03_Odd_Even
Connections:
- net at PS3.4 (-VOUT): now also J4.6 (Pin_6)
- net at PS3.5 (+VOUT): now also J4.5 (Pin_5)
- net at PS1.2 (-VOUT): now also J4.2 (Pin_2)
- net at PS1.3 (+VOUT): now also J4.1 (Pin_1)
- net at PS2.4 (-VOUT): now also J4.4 (Pin_4)
- net at PS2.5 (+VOUT): now also J4.3 (Pin_3)
- no-connect marks 4 -> 0
